File: cad/button/button.sch (KiCad schematic (older format))
At the start: 31 parts, among them J1 Ali_uSD_SPI, J2 SWD, Q1 DMC2038LVT, SW1 Button, U1 STM32L072KZTx, U2 PAM8302AAS

Commit message: move to kicad 5 footprints
Parts:
- C1, C10, C11, C2, C3, C4, C5, C6, C7, C8, C9: footprint Capacitors_SMD:C_0603_HandSoldering -> Capacitor_SMD:C_0603_1608Metric_Pad1.05x0.95mm_HandSolder
- FB1, FB2: footprint Resistors_SMD:R_0603_HandSoldering -> Inductor_SMD:L_0603_1608Metric_Pad1.05x0.95mm_HandSolder
- Q1: footprint TO_SOT_Packages_SMD:TSOT-23-6 -> Package_TO_SOT_SMD:TSOT-23-6_HandSoldering
- R1, R2, R3, R4, R5, R6, R7, R8, R9: footprint Resistors_SMD:R_0603_HandSoldering -> Resistor_SMD:R_0603_1608Metric_Pad1.05x0.95mm_HandSolder
- U1: footprint Housings_QFP:LQFP-32_7x7mm_Pitch0.8mm -> Package_QFP:LQFP-32_7x7mm_P0.8mm
- U2: footprint Housings_SSOP:MSOP-8_3x3mm_Pitch0.65mm -> Package_SO:MSOP-8_3x3mm_P0.65mm
Changed lines of the file:
@@
 F 0 "U1" H 3000 6200 50  0000 C CNN
 F 1 "STM32L072KZTx" H 2950 6100 50  0000 C CNN
-F 2 "Housings_QFP:LQFP-32_7x7mm_Pitch0.8mm" H 2600 4900 50  0001 R CNN
+F 2 "Package_QFP:LQFP-32_7x7mm_P0.8mm" H 2600 4900 50  0001 R CNN
 F 3 "http://www.st.com/st-web-ui/static/active/en/resource/technical/document/datasheet/DM00141133.pdf" H 3100 5800 50  0001 C CNN
 	1    3100 5800
@@
 F 0 "U2" H 7000 2900 50  0000 C CNN
 F 1 "PAM8302AAS" H 6800 2800 50  0000 L CNN
-F 2 "Housings_SSOP:MSOP-8_3x3mm_Pitch0.65mm" H 7350 2350 50  0001 C CNN
+F 2 "Package_SO:MSOP-8_3x3mm_P0.65mm" H 7350 2350 50  0001 C CNN
 F 3 "https://www.diodes.com/assets/Datasheets/PAM8302A.pdf" H 7350 2350 50  0001 C CNN
 	1    7350 2350
@@
 F 0 "C6" V 3300 4700 50  0000 L CNN
 F 1 "100nF" V 3400 4700 50  0000 L CNN
-F 2 "Capacitors_SMD:C_0603_HandSoldering" H 3350 4550 50  0001 C CNN
+F 2 "Capacitor_SMD:C_0603_1608Metric_Pad1.05x0.95mm_HandSolder" H 3350 4550 50  0001 C CNN
 F 3 "~" H 3350 4550 50  0001 C CNN
 	1    3350 4550
@@
 F 0 "C3" V 2800 4600 50  0000 R CNN
 F 1 "100nF" V 2900 4750 50  0000 R CNN
-F 2 "Capacitors_SMD:C_0603_HandSoldering" H 2850 4350 50  0001 C CNN
+F 2 "Capacitor_SMD:C_0603_1608Metric_Pad1.05x0.95mm_HandSolder" H 2850 4350 50  0001 C CNN
 F 3 "~" H 2850 4350 50  0001 C CNN
 	1    2850 4350
@@
 F 0 "C4" V 2800 4800 50  0000 R CNN
 F 1 "100nF" V 2900 4950 50  0000 R CNN
-F 2 "Capacitors_SMD:C_0603_HandSoldering" H 2850 4550 50  0001 C CNN
+F 2 "Capacitor_SMD:C_0603_1608Metric_Pad1.05x0.95mm_HandSolder" H 2850 4550 50  0001 C CNN
 F 3 "~" H 2850 4550 50  0001 C CNN
 	1    2850 4550
@@
 F 0 "R5" H 2109 5496 50  0000 L CNN
 F 1 "10K" H 2109 5405 50  0000 L CNN
-F 2 "Resistors_SMD:R_0603_HandSoldering" H 2050 5450 50  0001 C CNN
+F 2 "Resistor_SMD:R_0603_1608Metric_Pad1.05x0.95mm_HandSolder" H 2050 5450 50  0001 C CNN
 F 3 "~" H 2050 5450 50  0001 C CNN
 	1    2050 5450
@@
 F 0 "R9" V 6950 2800 50  0000 C CNN
 F 1 "10K" V 6850 2800 50  0000 C CNN
-F 2 "Resistors_SMD:R_0603_HandSoldering" H 7050 2800 50  0001 C CNN
+F 2 "Resistor_SMD:R_0603_1608Metric_Pad1.05x0.95mm_HandSolder" H 7050 2800 50  0001 C CNN
 F 3 "~" H 7050 2800 50  0001 C CNN
 	1    7050 2800
@@
 F 0 "Q1" H 4150 2550 50  0000 R CNN
 F 1 "DMC2038LVT" H 4450 2450 50  0000 R CNN
-F 2 "TO_SOT_Packages_SMD:TSOT-23-6" H 3950 2425 50  0001 L CNN
+F 2 "Package_TO_SOT_SMD:TSOT-23-6_HandSoldering" H 3950 2425 50  0001 L CNN
 F 3 "https://www.mouser.de/datasheet/2/115/DMC2038LVT-82505.pdf" H 3950 2350 50  0001 L CNN
 	1    3750 2500
@@
 F 0 "Q1" V 4000 1750 50  0000 C CNN
 F 1 "DMC2038LVT" V 3900 1750 50  0000 C CNN
-F 2 "TO_SOT_Packages_SMD:TSOT-23-6" H 3850 1675 50  0001 L CNN
+F 2 "Package_TO_SOT_SMD:TSOT-23-6_HandSoldering" H 3850 1675 50  0001 L CNN
 F 3 "https://www.mouser.de/datasheet/2/115/DMC2038LVT-82505.pdf" H 3850 1600 50  0001 L CNN
 	2    3650 1750
@@
 F 0 "C2" V 2800 4000 50  0000 R CNN
 F 1 "10uF" V 2900 4000 50  0000 R CNN
-F 2 "Capacitors_SMD:C_0603_HandSoldering" H 2850 4150 50  0001 C CNN
+F 2 "Capacitor_SMD:C_0603_1608Metric_Pad1.05x0.95mm_HandSolder" H 2850 4150 50  0001 C CNN
 F 3 "~" H 2850 4150 50  0001 C CNN
 	1    2850 4150
@@
 F 0 "C5" V 3300 4500 50  0000 L CNN
 F 1 "1uF" V 3400 4500 50  0000 L CNN
-F 2 "Capacitors_SMD:C_0603_HandSoldering" H 3350 4350 50  0001 C CNN
+F 2 "Capacitor_SMD:C_0603_1608Metric_Pad1.05x0.95mm_HandSolder" H 3350 4350 50  0001 C CNN
 F 3 "~" H 3350 4350 50  0001 C CNN
 	1    3350 4350
@@
 F 0 "R1" V 3204 2050 50  0000 C CNN
 F 1 "10K" V 3295 2050 50  0000 C CNN
-F 2 "Resistors_SMD:R_0603_HandSoldering" H 3400 2050 50  0001 C CNN
+F 2 "Resistor_SMD:R_0603_1608Metric_Pad1.05x0.95mm_HandSolder" H 3400 2050 50  0001 C CNN
 F 3 "~" H 3400 2050 50  0001 C CNN
 	1    3400 2050
@@
 F 0 "R3" H 4259 2096 50  0000 L CNN
 F 1 "not fitted" H 4259 2005 50  0000 L CNN
-F 2 "Resistors_SMD:R_0603_HandSoldering" H 4200 2050 50  0001 C CNN
+F 2 "Resistor_SMD:R_0603_1608Metric_Pad1.05x0.95mm_HandSolder" H 4200 2050 50  0001 C CNN
 F 3 "~" H 4200 2050 50  0001 C CNN
 	1    4200 2050
@@
 F 0 "R2" H 4259 2746 50  0000 L CNN
 F 1 "10K" H 4259 2655 50  0000 L CNN
-F 2 "Resistors_SMD:R_0603_HandSoldering" H 4200 2700 50  0001 C CNN
+F 2 "Resistor_SMD:R_0603_1608Metric_Pad1.05x0.95mm_HandSolder" H 4200 2700 50  0001 C CNN
 F 3 "~" H 4200 2700 50  0001 C CNN
 	1    4200 2700
@@
 F 0 "C1" H 2450 2300 50  0000 R CNN
 F 1 "10uF" H 2450 2200 50  0000 R CNN
-F 2 "Capacitors_SMD:C_0603_HandSoldering" H 2550 2250 50  0001 C CNN
+F 2 "Capacitor_SMD:C_0603_1608Metric_Pad1.05x0.95mm_HandSolder" H 2550 2250 50  0001 C CNN
 F 3 "~" H 2550 2250 50  0001 C CNN
 	1    2550 2250
@@
 F 0 "R4" H 3259 4196 50  0000 L CNN
 F 1 "10" H 3259 4105 50  0000 L CNN
-F 2 "Resistors_SMD:R_0603_HandSoldering" H 3200 4150 50  0001 C CNN
+F 2 "Resistor_SMD:R_0603_1608Metric_Pad1.05x0.95mm_HandSolder" H 3200 4150 50  0001 C CNN
 F 3 "~" H 3200 4150 50  0001 C CNN
 	1    3200 4150
@@
 F 0 "C10" H 8050 2750 50  0000 L CNN
 F 1 "220pF" H 8000 2650 50  0000 L CNN
-F 2 "Capacitors_SMD:C_0603_HandSoldering" H 8350 2700 50  0001 C CNN
+F 2 "Capacitor_SMD:C_0603_1608Metric_Pad1.05x0.95mm_HandSolder" H 8350 2700 50  0001 C CNN
 F 3 "~" H 8350 2700 50  0001 C CNN
 	1    8350 2700
@@
 F 0 "C11" H 8650 2750 50  0000 L CNN
 F 1 "220pF" H 8650 2650 50  0000 L CNN
-F 2 "Capacitors_SMD:C_0603_HandSoldering" H 8550 2700 50  0001 C CNN
+F 2 "Capacitor_SMD:C_0603_1608Metric_Pad1.05x0.95mm_HandSolder" H 8550 2700 50  0001 C CNN
 F 3 "~" H 8550 2700 50  0001 C CNN
 	1    8550 2700
@@
 F 0 "FB1" V 8045 2150 50  0000 C CNN
 F 1 "Ferrite_Bead_Small" V 8046 2150 50  0001 C CNN
-F 2 "Resistors_SMD:R_0603_HandSoldering" V 7830 2150 50  0001 C CNN
+F 2 "Inductor_SMD:L_0603_1608Metric_Pad1.05x0.95mm_HandSolder" V 7830 2150 50  0001 C CNN
 F 3 "~" H 7900 2150 50  0001 C CNN
 	1    7900 2150
@@
 F 0 "FB2" V 7750 2350 50  0000 C CNN
 F 1 "Ferrite_Bead_Small" V 8046 2350 50  0001 C CNN
-F 2 "Resistors_SMD:R_0603_HandSoldering" V 7830 2350 50  0001 C CNN
+F 2 "Inductor_SMD:L_0603_1608Metric_Pad1.05x0.95mm_HandSolder" V 7830 2350 50  0001 C CNN
 F 3 "~" H 7900 2350 50  0001 C CNN
 	1    7900 2350
@@
 F 0 "C9" V 7750 1600 50  0000 L CNN
 F 1 "10uF" V 7850 1550 50  0000 L CNN
-F 2 "Capacitors_SMD:C_0603_HandSoldering" H 7600 1650 50  0001 C CNN
+F 2 "Capacitor_SMD:C_0603_1608Metric_Pad1.05x0.95mm_HandSolder" H 7600 1650 50  0001 C CNN
 F 3 "~" H 7600 1650 50  0001 C CNN
 	1    7600 1650
@@
 F 0 "C7" V 6000 2150 50  0000 C CNN
 F 1 "1uF" V 6100 2150 50  0000 C CNN
-F 2 "Capacitors_SMD:C_0603_HandSoldering" H 6250 2150 50  0001 C CNN
+F 2 "Capacitor_SMD:C_0603_1608Metric_Pad1.05x0.95mm_HandSolder" H 6250 2150 50  0001 C CNN
 F 3 "~" H 6250 2150 50  0001 C CNN
 	1    6250 2150
@@
 F 0 "C8" V 6400 2350 50  0000 C CNN
 F 1 "1uF" V 6500 2350 50  0000 C CNN
-F 2 "Capacitors_SMD:C_0603_HandSoldering" H 6250 2350 50  0001 C CNN
+F 2 "Capacitor_SMD:C_0603_1608Metric_Pad1.05x0.95mm_HandSolder" H 6250 2350 50  0001 C CNN
 F 3 "~" H 6250 2350 50  0001 C CNN
 	1    6250 2350
@@
 F 0 "R7" V 6300 2150 50  0000 C CNN
 F 1 "10K" V 6400 2150 50  0000 C CNN
-F 2 "Resistors_SMD:R_0603_HandSoldering" H 6550 2150 50  0001 C CNN
+F 2 "Resistor_SMD:R_0603_1608Metric_Pad1.05x0.95mm_HandSolder" H 6550 2150 50  0001 C CNN
 F 3 "~" H 6550 2150 50  0001 C CNN
 	1    6550 2150
@@
 F 0 "R8" V 6700 2350 50  0000 C CNN
 F 1 "10K" V 6800 2350 50  0000 C CNN
-F 2 "Resistors_SMD:R_0603_HandSoldering" H 6550 2350 50  0001 C CNN
+F 2 "Resistor_SMD:R_0603_1608Metric_Pad1.05x0.95mm_HandSolder" H 6550 2350 50  0001 C CNN
 F 3 "~" H 6550 2350 50  0001 C CNN
 	1    6550 2350
@@
 F 0 "R6" V 3800 5050 50  0000 L CNN
 F 1 "1K" V 4000 5050 50  0000 L CNN
-F 2 "Resistors_SMD:R_0603_HandSoldering" H 3900 5100 50  0001 C CNN
+F 2 "Resistor_SMD:R_0603_1608Metric_Pad1.05x0.95mm_HandSolder" H 3900 5100 50  0001 C CNN
 F 3 "~" H 3900 5100 50  0001 C CNN
 	1    3900 5100
